Commit message: feat: may3 version, refine inertia for revo3

File: revo3_system/urdf/revo3_left.urdf (robot description, URDF)
Before this commit: robot revo3_single, 29 links, 28 joints
Links:
- link left_index_DIP_Link: mass 0.01 -> 0.008
- link left_index_PIP_Link: mass 0.0332 -> 0.031
- link left_middle_MPR_Link: mass 0.013 -> 0.012
- link left_middle_PIP_Link: mass 0.0332 -> 0.031

File: revoarm_system/urdf/revoarm_bimanual_revo3.urdf (robot description, URDF)
Before this commit: robot revoarm_bimanual, 78 links, 77 joints
Links:
- link left_index_DIP_Link: mass 0.01 -> 0.008
- link left_index_PIP_Link: mass 0.0332 -> 0.031
- link left_middle_MPR_Link: mass 0.013 -> 0.012
- link left_middle_PIP_Link: mass 0.0332 -> 0.031

File: revoarm_system/urdf/revoarm_single_left_revo3.urdf (robot description, URDF)
Before this commit: robot revoarm_single, 39 links, 38 joints
Links:
- link left_index_DIP_Link: mass 0.01 -> 0.008
- link left_index_PIP_Link: mass 0.0332 -> 0.031
- link left_middle_MPR_Link: mass 0.013 -> 0.012
- link left_middle_PIP_Link: mass 0.0332 -> 0.031

File: revotron_system/urdf/revotron_bimanual_revo3.urdf (robot description, URDF)
Before this commit: robot revotron_bimanual, 78 links, 77 joints
Links:
- link left_index_DIP_Link: mass 0.01 -> 0.008
- link left_index_PIP_Link: mass 0.0332 -> 0.031
- link left_middle_MPR_Link: mass 0.013 -> 0.012
- link left_middle_PIP_Link: mass 0.0332 -> 0.031
