Commit message: refine: update revo3 hand inertia values and zero out tip link masses
Recalculated inertia tensors for all finger links and set tip link
inertia/mass to zero since they are fixed joints.

Co-Authored-By: Claude Opus 4.7 (1M context) <noreply@anthropic.com>

File: revo3_system/urdf/revo3_right.urdf (robot description, URDF)
Before this commit: robot revo3_single, 29 links, 28 joints
Links:
- link right_index_tip_Link: mass 0.001 -> 0
- link right_little_tip_Link: mass 0.001 -> 0
- link right_middle_tip_Link: mass 0.001 -> 0
- link right_palm: mass 0.001 -> 0.00
- link right_ring_tip_Link: mass 0.001 -> 0
- link right_thumb_tip_Link: mass 0.001 -> 0
