Commit message: fix: revo2/revo3 +revoarm_single bugs

File: revoarm_system/urdf/revoarm_bimanual_revo3.urdf (robot description, URDF)
Before this commit: robot revoarm_bimanual, 78 links, 77 joints
Joints:
- joint left_connector_tip_joint: origin xyz=0.0 0.0 -0.0 rpy=0 3.14 3.14 -> xyz=0.0 0.0 0.0 rpy=0 3.14 3.14

File: revoarm_system/urdf/revoarm_single_left_revo2.urdf (robot description, URDF)
Before this commit: robot revoarm_single, 33 links, 32 joints
Joints:
- joint left_connector_tip_joint: origin xyz=0.0000760 0.0001518 -0.0583 rpy=0 3.14 -1.57 -> xyz=0.0000760 0.0001518 -0.0583 rpy=0 3.14 0
- joint left_hand_base_joint: origin xyz=0 0 0 rpy=0 0 0 -> xyz=0 0 -0.0118 rpy=0 0 0

File: revoarm_system/urdf/revoarm_single_left_revo3.urdf (robot description, URDF)
Before this commit: robot revoarm_single, 39 links, 38 joints
Joints:
- joint left_connector_tip_joint: origin xyz=0.0 0.0 -0.0 rpy=0 3.14 3.14 -> xyz=0.0 0.0 0.0 rpy=0 3.14 0
- joint left_hand_base_joint: origin xyz=0 0 0 rpy=0 0 0 -> xyz=0 0 -0.0118 rpy=0 0 0

File: revoarm_system/urdf/revoarm_single_right_revo2.urdf (robot description, URDF)
Before this commit: robot revoarm_single, 33 links, 32 joints
Joints:
- joint right_connector_tip_joint: origin xyz=0.0000760 -0.0001518 -0.0583 rpy=0 3.14 1.57 -> xyz=0.0000760 -0.0001518 -0.0583 rpy=0 3.14 0
- joint right_hand_base_joint: origin xyz=0 0 0 rpy=0 0 0 -> xyz=0 0 -0.0118 rpy=0 0 0

File: revoarm_system/urdf/revoarm_single_right_revo3.urdf (robot description, URDF)
Before this commit: robot revoarm_single, 39 links, 38 joints
Joints:
- joint right_hand_base_joint: origin xyz=0 0 0 rpy=0 0 0 -> xyz=0 0 -0.0118 rpy=0 0 0
